Commit message: Added imu offset from ideal with measurements

File: src/localization/urdf/bot.xacro (robot description, xacro)
@@ -6,4 +6,7 @@
     <xacro:property name="back_thickness" value="0.00625" />
     <xacro:property name="rad_per_deg" value="${pi/180}" />
+    <xacro:property name="imu_roll" value="2.9" />
+    <xacro:property name="imu_pitch" value="0.6" />
+    <xacro:property name="imu_yaw" value="-1.0" />
     <xacro:macro name="material">
         <material name="Grey">
@@ -42,11 +45,21 @@
     </link>
     <link name="mpu"/>
+    <link name="ideal_mpu"/>
     <joint name="mpu_frame" type="fixed">
-        <origin xyz="${back_thickness/2 - 0.037 + 0.0375 - 0.002} 0.01 0.157" rpy="${1 * rad_per_deg} ${pi/2 - 0 * rad_per_deg} ${pi + 2 * rad_per_deg}" />
+        <origin
+            xyz="${back_thickness/2 - 0.037 + 0.0375 - 0.002} 0.01 0.157"
+            rpy="${0} ${pi/2} ${pi}" />
         <parent link="body" />
-        <child link="mpu" />
+        <child link="ideal_mpu" />
     </joint>
     <!-- 0.157 m above the center
     0.002286 m off center
     37.5 cm in front of the back, the board is 1.5 mm thick -->
+    <joint name="mpu_offset" type="fixed">
+        <origin
+            xyz="0 0 0"
+            rpy="${imu_roll * rad_per_deg} ${imu_pitch * rad_per_deg} ${imu_yaw * rad_per_deg}" />
+        <parent link="ideal_mpu" />
+        <child link="mpu" />
+    </joint>
 </robot>

Commit message: Moved robot state publishing to launch file

File: src/localization/urdf/bot.xacro (robot description, xacro)
@@ -6,7 +6,7 @@
     <xacro:property name="back_thickness" value="0.00625" />
     <xacro:property name="rad_per_deg" value="${pi/180}" />
-    <xacro:property name="imu_roll" value="2.9" />
-    <xacro:property name="imu_pitch" value="0.6" />
-    <xacro:property name="imu_yaw" value="-1.0" />
+    <xacro:property name="mpu_roll" value="2.9" />
+    <xacro:property name="mpu_pitch" value="0.6" />
+    <xacro:property name="mpu_yaw" value="-1.0" />
     <xacro:macro name="material">
         <material name="Grey">
@@ -46,20 +46,20 @@
     <link name="mpu"/>
     <link name="ideal_mpu"/>
-    <joint name="mpu_frame" type="fixed">
+    <joint name="body_to_ideal_mpu" type="fixed">
+        <parent link="body" />
+        <child link="ideal_mpu" />
         <origin
             xyz="${back_thickness/2 - 0.037 + 0.0375 - 0.002} 0.01 0.157"
             rpy="${0} ${pi/2} ${pi}" />
-        <parent link="body" />
-        <child link="ideal_mpu" />
     </joint>
     <!-- 0.157 m above the center
     0.002286 m off center
     37.5 cm in front of the back, the board is 1.5 mm thick -->
-    <joint name="mpu_offset" type="fixed">
+    <joint name="ideal_mpu_to_mpu" type="fixed">
+        <parent link="body" />
+        <child link="mpu" />
         <origin
             xyz="0 0 0"
-            rpy="${imu_roll * rad_per_deg} ${imu_pitch * rad_per_deg} ${imu_yaw * rad_per_deg}" />
-        <parent link="ideal_mpu" />
-        <child link="mpu" />
+            rpy="${mpu_roll * rad_per_deg} ${mpu_pitch * rad_per_deg} ${mpu_yaw * rad_per_deg}" />
     </joint>
 </robot>

Commit message: Corrected joint from ideal to mpu

File: src/localization/urdf/bot.xacro (robot description, xacro)
@@ -57,5 +57,5 @@
     37.5 cm in front of the back, the board is 1.5 mm thick -->
     <joint name="ideal_mpu_to_mpu" type="fixed">
-        <parent link="body" />
+        <parent link="ideal_mpu" />
         <child link="mpu" />
         <origin
